Commit message: feat(robot_description): Add Nerf launcher support and update Gazebo plugin
- Modify launch file to support optional Nerf launcher component
- Update Gazebo plugin from Ignition to gz-ros2-control
- Add new launch argument `include_nerf_launcher`
- Update package.xml to use generic ROS build type condition
- Improve URDF parameter handling with ParameterValue
- Prepare infrastructure for adding Nerf launcher component to robot XL

File: urdf/common/gazebo.urdf.xacro (robot description, xacro)
@@ -3,5 +3,6 @@
   <xacro:macro name="controller" params="config_file namespace:=''">
     <gazebo>
-      <plugin filename="ign_ros2_control-system" name="ign_ros2_control::IgnitionROS2ControlPlugin">
+      <!-- Gazebo (Ignition/ros_gz) ros2_control system plugin -->
+      <plugin filename="gz-ros2-control-system" name="gz_ros2_control::GazeboSimSystem">
         <parameters>${config_file}</parameters>
         <ros>

File: urdf/common/ros2_control.urdf.xacro (robot description, xacro)
@@ -23,5 +23,5 @@
     </ros2_control>
   </xacro:macro>
-  <xacro:macro name="robot_system" params="name:='robot_system' namespace:=''">
+  <xacro:macro name="robot_system" params="name:='robot_system' namespace:='' include_nerf:='False'">
     <xacro:property name="ns" value="${namespace + '/' if namespace != '' else ''}" />
     <ros2_control name="${ns}${name}" type="system">
@@ -55,7 +55,28 @@
         <state_interface name="velocity" />
       </joint>
+      <!-- Optional Nerf launcher joints (servos + ESCs) -->
+      <xacro:if value="${include_nerf}">
+        <!-- Pan/Tilt servos: position interfaces -->
+        <joint name="pan_servo_joint">
+          <command_interface name="position" />
+          <state_interface name="position" />
+        </joint>
+        <joint name="tilt_servo_joint">
+          <command_interface name="position" />
+          <state_interface name="position" />
+        </joint>
+        <!-- Flywheel ESCs: velocity interfaces (normalized or rad/s per HW) -->
+        <joint name="esc_left_joint">
+          <command_interface name="velocity" />
+          <state_interface name="velocity" />
+        </joint>
+        <joint name="esc_right_joint">
+          <command_interface name="velocity" />
+          <state_interface name="velocity" />
+        </joint>
+      </xacro:if>
     </ros2_control>
   </xacro:macro>
-  <xacro:macro name="gz_robot_system" params="name:='robot_system' namespace:=''">
+  <xacro:macro name="gz_robot_system" params="name:='robot_system' namespace:='' include_nerf:='False'">
     <xacro:property name="ns" value="${namespace + '/' if namespace != '' else ''}" />
     <ros2_control name="${ns}${name}" type="system">
@@ -86,4 +107,23 @@
         <state_interface name="velocity" />
       </joint>
+      <!-- Optional Nerf launcher joints for simulation -->
+      <xacro:if value="${include_nerf}">
+        <joint name="pan_servo_joint">
+          <command_interface name="position" />
+          <state_interface name="position" />
+        </joint>
+        <joint name="tilt_servo_joint">
+          <command_interface name="position" />
+          <state_interface name="position" />
+        </joint>
+        <joint name="esc_left_joint">
+          <command_interface name="velocity" />
+          <state_interface name="velocity" />
+        </joint>
+        <joint name="esc_right_joint">
+          <command_interface name="velocity" />
+          <state_interface name="velocity" />
+        </joint>
+      </xacro:if>
       <sensor name="${ns}imu">
         <state_interface name="orientation.x" />

File: urdf/robot_xl.urdf.xacro (robot description, xacro)
@@ -6,4 +6,5 @@
   <xacro:arg name="controller_config" default="" />
   <xacro:arg name="include_camera_mount" default="false" />
+  <xacro:arg name="include_nerf_launcher" default="false" />
   <xacro:arg name="manipulator_serial_port" default="/dev/ttyUSB0" />
   <xacro:arg name="mecanum" default="false" />
@@ -12,5 +13,6 @@
   <xacro:include filename="$(find robot_description)/urdf/robot_xl/robot_xl_macro.urdf.xacro" ns="husarion" />
   <xacro:include filename="$(find husarion_components_description)/urdf/components.urdf.xacro" ns="components" />
-  <xacro:husarion.robot_xl controller_config="$(arg controller_config)" include_camera_mount="$(arg include_camera_mount)" mecanum="$(arg mecanum)" namespace="$(arg namespace)" use_sim="$(arg use_sim)" />
+  <!-- <xacro:husarion.robot_xl controller_config="$(arg controller_config)" include_camera_mount="$(arg include_camera_mount)" mecanum="$(arg mecanum)" namespace="$(arg namespace)" use_sim="$(arg use_sim)" /> -->
+  <xacro:husarion.robot_xl controller_config="$(arg controller_config)" include_camera_mount="$(arg include_camera_mount)" include_nerf_launcher="$(arg include_nerf_launcher)" mecanum="$(arg mecanum)" namespace="$(arg namespace)" use_sim="$(arg use_sim)" />
   <xacro:components.create_components components_config_path="$(arg components_config)" namespace="" use_sim="$(arg use_sim)" />
   <xacro:if value="${'$(arg configuration)'.startswith('manipulation')}">

File: urdf/robot_xl/rosbot_xl_macro.urdf.xacro (robot description, xacro)
@@ -3,4 +3,5 @@
   <xacro:macro name="robot_xl" params="controller_config
             include_camera_mount
+            include_nerf_launcher
             mecanum
             namespace
@@ -16,4 +17,5 @@
     <xacro:include filename="$(find robot_description)/urdf/robot_xl/wheel.urdf.xacro" ns="wheel" />
     <xacro:include filename="$(find robot_description)/urdf/robot_xl/components/camera_mount.urdf.xacro" ns="camera_mount" />
+    <xacro:include filename="$(find robot_description)/urdf/robot_xl/components/nerf_launcher.urdf.xacro" ns="nerf_launcher" />
     <!-- BODY -->
     <xacro:body.body wheel_radius="${wheel_radius}" />
@@ -21,4 +23,8 @@
     <xacro:if value="${include_camera_mount}">
       <xacro:camera_mount.camera_mount parent_link="cover_link" xyz="-0.1 0.0 0.0" />
+    </xacro:if>
+    <!-- Optional NERF launcher component -->
+    <xacro:if value="${include_nerf_launcher}">
+      <xacro:nerf_launcher.nerf_launcher parent_link="cover_link" xyz="0.08 0.0 0.02" />
     </xacro:if>
     <!-- WHEEL -->
@@ -30,9 +36,9 @@
     <xacro:unless value="${use_sim}">
       <xacro:ros2_control.imu namespace="${namespace}" />
-      <xacro:ros2_control.robot_system namespace="${namespace}" />
+      <xacro:ros2_control.robot_system namespace="${namespace}" include_nerf="${include_nerf_launcher}" />
     </xacro:unless>
     <!-- GAZEBO PLUGINS -->
     <xacro:if value="${use_sim}">
-      <xacro:ros2_control.gz_robot_system namespace="${namespace}" />
+      <xacro:ros2_control.gz_robot_system namespace="${namespace}" include_nerf="${include_nerf_launcher}" />
       <xacro:gazebo.controller config_file="${controller_config}" namespace="${namespace}" />
       <xacro:gazebo.imu reference_frame="imu_link" namespace="${namespace}" />
