Commit message: feat(robot_description): Refactor robot_xl macro with comprehensive configuration options
- Add flexible macro for robot_xl with configurable parameters
- Include optional components like camera mount and Nerf launcher
- Support mecanum and standard wheel configurations
- Add namespace and simulation mode parameters
- Implement conditional loading of hardware and simulation plugins
- Remove previous wrapper macro and replace with full implementation
- Enable dynamic configuration of robot components through macro parameters

File: urdf/robot_xl/robot_xl_macro.urdf.xacro (robot description, xacro)
@@ -1,9 +1,50 @@
 <?xml version='1.0'?>
 <robot xmlns:xacro="http://wiki.ros.org/xacro">
-        <!--
-    Wrapper macro to provide the expected filename for installed xacro includes.
-    This simply includes the existing robot_xl_macro.urdf.xacro so both source
-    and installed-time includes that reference robot_xl_macro.urdf.xacro will work.
-  -->
-        <xacro:include filename="$(find robot_description)/urdf/robot_xl/robot_xl_macro.urdf.xacro" />
+  <xacro:macro name="robot_xl" params="controller_config
+            include_camera_mount
+            include_nerf_launcher
+            mecanum
+            namespace
+            use_sim">
+    <!-- PROPERTIES -->
+    <xacro:property name="wheel_radius" value="${0.05 if mecanum else 0.048}" />
+    <!-- INCLUDE ROBOT MACRO -->
+    <xacro:include filename="$(find robot_description)/urdf/common/gazebo.urdf.xacro" ns="gazebo" />
+    <xacro:include filename="$(find robot_description)/urdf/common/ros2_control.urdf.xacro" ns="ros2_control" />
+    <!-- <xacro:include filename="$(find robot_description)/urdf/common/webots.urdf.xacro" ns="webots" /> -->
+    <xacro:include filename="$(find robot_description)/urdf/robot_xl/body.urdf.xacro" ns="body" />
+    <xacro:include filename="$(find robot_description)/urdf/robot_xl/components/antenna.urdf.xacro" ns="antenna" />
+    <xacro:include filename="$(find robot_description)/urdf/robot_xl/wheel.urdf.xacro" ns="wheel" />
+    <xacro:include filename="$(find robot_description)/urdf/robot_xl/components/camera_mount.urdf.xacro" ns="camera_mount" />
+    <xacro:include filename="$(find robot_description)/urdf/robot_xl/components/nerf_launcher.urdf.xacro" ns="nerf_launcher" />
+    <!-- BODY -->
+    <xacro:body.body wheel_radius="${wheel_radius}" />
+    <xacro:antenna.antenna parent_link="cover_link" xyz="-0.155 -0.055 -0.02" rpy="-0.4 0.0 0.0" antenna_angle="0.3" />
+    <xacro:if value="${include_camera_mount}">
+      <xacro:camera_mount.camera_mount parent_link="cover_link" xyz="-0.1 0.0 0.0" />
+    </xacro:if>
+    <!-- Optional NERF launcher component -->
+    <xacro:if value="${include_nerf_launcher}">
+      <xacro:nerf_launcher.nerf_launcher parent_link="cover_link" xyz="0.08 0.0 0.02" launcher_angle="-0.15" />
+    </xacro:if>
+    <!-- WHEEL -->
+    <xacro:wheel.wheel wheel_radius="${wheel_radius}" side="fl" mecanum="${mecanum}" />
+    <xacro:wheel.wheel wheel_radius="${wheel_radius}" side="fr" mecanum="${mecanum}" />
+    <xacro:wheel.wheel wheel_radius="${wheel_radius}" side="rl" mecanum="${mecanum}" />
+    <xacro:wheel.wheel wheel_radius="${wheel_radius}" side="rr" mecanum="${mecanum}" />
+    <!-- HARDWARE PLUGINS -->
+    <xacro:unless value="${use_sim}">
+      <xacro:ros2_control.imu namespace="${namespace}" />
+      <xacro:ros2_control.robot_system namespace="${namespace}" include_nerf="${include_nerf_launcher}" />
+    </xacro:unless>
+    <!-- GAZEBO PLUGINS -->
+    <xacro:if value="${use_sim}">
+      <xacro:ros2_control.gz_robot_system namespace="${namespace}" include_nerf="${include_nerf_launcher}" />
+      <xacro:gazebo.controller config_file="${controller_config}" namespace="${namespace}" />
+      <xacro:gazebo.imu reference_frame="imu_link" namespace="${namespace}" />
+      <!-- <xacro:if value="${simulation_engine == 'webots'}">
+        <xacro:webots.controller />
+      </xacro:if> -->
+    </xacro:if>
+  </xacro:macro>
 </robot>
